Commit message: Updated model

File: darwinOP.urdf (robot description, URDF)
Before this commit: robot darwinOP, 30 links, 29 joints
Links:
- link MP_ANKLE1_L: geometry collision mesh filename=package://darwinOP/meshes/ankle1_l_coll.stl scale=1 1 1; visual mesh filename=package://darwinOP/meshes/ankle1_l.STL scale=1 1 1
- link MP_ANKLE1_R: geometry collision mesh filename=package://darwinOP/meshes/ankle1_r_coll.stl scale=1 1 1; visual mesh filename=package://darwinOP/meshes/ankle1_r.STL scale=1 1 1
- link MP_ANKLE2_L: mass 0.16710792 -> 0.0794462; geometry collision mesh filename=package://darwinOP/meshes/ankle2_l_coll.stl scale=1 1 1; visual mesh filename=package://darwinOP/meshes/ankle2_l.STL scale=1 1 1
- link MP_ANKLE2_R: mass 0.16710792 -> 0.0794462; geometry collision mesh filename=package://darwinOP/meshes/ankle2_r_coll.stl scale=1 1 1; visual mesh filename=package://darwinOP/meshes/ankle2_r.STL scale=1 1 1
- link MP_ARM_GRIPPER_MOV_L: geometry collision box size=0.002 0.01 0.032; collision box size=0.032 0.005 0.032
- link MP_ARM_GRIPPER_MOV_R: geometry collision box size=0.002 0.01 0.032; collision box size=0.032 0.005 0.032
- link MP_ARM_HIGH_L: geometry collision mesh filename=package://darwinOP/meshes/arm_high_l_coll.stl scale=1 1 1; visual mesh filename=package://darwinOP/meshes/arm_high_l.STL scale=1 1 1
- link MP_ARM_HIGH_R: geometry collision mesh filename=package://darwinOP/meshes/arm_high_r_coll.stl scale=1 1 1; visual mesh filename=package://darwinOP/meshes/arm_high_r.STL scale=1 1 1
- link MP_ARM_LOW_L: mass 0.010 -> 0.059288504
- link MP_ARM_LOW_R: mass 0.010 -> 0.059288504; geometry collision box size=0.032 0.032 0.035; visual box size=0.032 0.032 0.035
- link MP_BACK_L: geometry collision box scale=1 1 1 size=0.001 0.001 0.001; visual box scale=1 1 1 size=0.001 0.001 0.001
- link MP_BODY: geometry collision mesh filename=package://darwinOP/meshes/body_coll.stl scale=1 1 1; visual mesh filename=package://darwinOP/meshes/body.STL scale=1 1 1
- link MP_HEAD: geometry collision mesh filename=package://darwinOP/meshes/head_coll.stl scale=1 1 1; visual mesh filename=package://darwinOP/meshes/head.STL scale=1 1 1
- link MP_NECK: geometry collision mesh filename=package://darwinOP/meshes/neck_coll.stl scale=1 1 1; visual mesh filename=package://darwinOP/meshes/neck.STL scale=1 1 1
- link MP_PELVIS_L: mass 0.197 -> 0.167; geometry collision mesh filename=package://darwinOP/meshes/pelvis_l_coll.stl scale=1 1 1; visual mesh filename=package://darwinOP/meshes/pelvis_l.STL scale=1 1 1
- link MP_PELVIS_R: geometry collision mesh filename=package://darwinOP/meshes/pelvis_r_coll.stl scale=1 1 1; visual mesh filename=package://darwinOP/meshes/pelvis_r.STL scale=1 1 1
- link MP_SHOULDER_L: geometry collision mesh filename=package://darwinOP/meshes/shoulder_l_coll.stl scale=1 1 1; visual mesh filename=package://darwinOP/meshes/shoulder_l.STL scale=1 1 1
- link MP_SHOULDER_R: geometry collision mesh filename=package://darwinOP/meshes/shoulder_r_coll.stl scale=1 1 1; visual mesh filename=package://darwinOP/meshes/shoulder_r.STL scale=1 1 1
- link MP_THIGH1_L: geometry collision mesh filename=package://darwinOP/meshes/thigh1_l_coll.stl scale=1 1 1; visual mesh filename=package://darwinOP/meshes/thigh1_l.STL scale=1 1 1
- link MP_THIGH1_R: geometry collision mesh filename=package://darwinOP/meshes/thigh1_r_coll.stl scale=1 1 1; visual mesh filename=package://darwinOP/meshes/thigh1_r.STL scale=1 1 1
- link MP_THIGH2_L: geometry collision mesh filename=package://darwinOP/meshes/thigh2_l_coll.stl scale=1 1 1; visual mesh filename=package://darwinOP/meshes/thigh2_l.STL scale=1 1 1
- link MP_THIGH2_R: geometry collision mesh filename=package://darwinOP/meshes/thigh2_r_coll.stl scale=1 1 1; visual mesh filename=package://darwinOP/meshes/thigh2_r.STL scale=1 1 1
- link MP_TIBIA_L: geometry collision mesh filename=package://darwinOP/meshes/tibia_l_coll.stl scale=1 1 1; visual mesh filename=package://darwinOP/meshes/tibia_l.STL scale=1 1 1
- link MP_TIBIA_R: mass 0.70309794 -> 0.070309794; geometry collision mesh filename=package://darwinOP/meshes/tibia_r_coll.stl scale=1 1 1; visual mesh filename=package://darwinOP/meshes/tibia_r.STL scale=1 1 1
Joints:
- joint j_gripper_l: origin xyz=0.048 0.01 0 rpy=0 0 0 -> xyz=0.048 0.01 0 rpy=0 0 1.0
- joint j_gripper_r: origin xyz=0.048 0.01 0 rpy=0 0 0 -> xyz=0.048 0.01 0 rpy=0 0 1.0
- joint j_high_arm_l: origin xyz=-0.016 0 0.02165 rpy=1.5707963 0.78539815 0 -> xyz=-0.016 0 0.02165 rpy=1.5707963 1.5707963 0
- joint j_high_arm_r: origin xyz=-0.016 0 0.02165 rpy=-1.5707963 0.78539815 0 -> xyz=0.016 0 0.02165 rpy=-1.5707963 1.5707963 0
- joint j_low_arm_l: origin xyz=-0.06 0 -0.016 rpy=-1.5707963 1.5707963 0 -> xyz=-0.06 0 -0.016 rpy=-1.5707963 3.14159 0
- joint j_low_arm_r: limit lower=-2.6179939 upper=2.6179939 effort=2.8 velocity=5.6548668 -> lower=-1.635 upper=2.6179939 effort=2.8 velocity=5.6548668; origin xyz=-0.06 0 -0.016 rpy=1.5707963 1.5707963 0 -> xyz=-0.06 0 0.016 rpy=-1.5707963 3.14159 0
- joint j_shoulder_r: origin xyz=0 0 0 rpy=0 0 1.5707963 -> xyz=0 0 0 rpy=0 0 -1.5707963

Commit message: updated the urdf

File: darwinOP.urdf (robot description, URDF)
Before this commit: robot darwinOP, 30 links, 29 joints
Links:
- link MP_ANKLE1_L: geometry collision mesh filename=package://Darwin_OP/meshes/ankle1_l_coll.stl scale=1 1 1; visual mesh filename=package://Darwin_OP/meshes/ankle1_l.STL scale=1 1 1
- link MP_ANKLE1_R: geometry collision mesh filename=package://Darwin_OP/meshes/ankle1_r_coll.stl scale=1 1 1; visual mesh filename=package://Darwin_OP/meshes/ankle1_r.STL scale=1 1 1
- link MP_ANKLE2_L: geometry collision mesh filename=package://Darwin_OP/meshes/ankle2_l_coll.stl scale=1 1 1; visual mesh filename=package://Darwin_OP/meshes/ankle2_l.STL scale=1 1 1
- link MP_ANKLE2_R: geometry collision mesh filename=package://Darwin_OP/meshes/ankle2_r_coll.stl scale=1 1 1; visual mesh filename=package://Darwin_OP/meshes/ankle2_r.STL scale=1 1 1
- link MP_ARM_HIGH_L: geometry collision mesh filename=package://Darwin_OP/meshes/arm_high_l_coll.stl scale=1 1 1; visual mesh filename=package://Darwin_OP/meshes/arm_high_l.STL scale=1 1 1
- link MP_ARM_HIGH_R: geometry collision mesh filename=package://Darwin_OP/meshes/arm_high_r_coll.stl scale=1 1 1; visual mesh filename=package://Darwin_OP/meshes/arm_high_r.STL scale=1 1 1
- link MP_BODY: geometry collision mesh filename=package://Darwin_OP/meshes/body_coll.stl scale=1 1 1; visual mesh filename=package://Darwin_OP/meshes/body.STL scale=1 1 1
- link MP_HEAD: geometry collision mesh filename=package://Darwin_OP/meshes/head_coll.stl scale=1 1 1; visual mesh filename=package://Darwin_OP/meshes/head.STL scale=1 1 1
- link MP_NECK: geometry collision mesh filename=package://Darwin_OP/meshes/neck_coll.stl scale=1 1 1; visual mesh filename=package://Darwin_OP/meshes/neck.STL scale=1 1 1
- link MP_PELVIS_L: geometry collision mesh filename=package://Darwin_OP/meshes/pelvis_l_coll.stl scale=1 1 1; visual mesh filename=package://Darwin_OP/meshes/pelvis_l.STL scale=1 1 1
- link MP_PELVIS_R: geometry collision mesh filename=package://Darwin_OP/meshes/pelvis_r_coll.stl scale=1 1 1; visual mesh filename=package://Darwin_OP/meshes/pelvis_r.STL scale=1 1 1
- link MP_SHOULDER_L: geometry collision mesh filename=package://Darwin_OP/meshes/shoulder_l_coll.stl scale=1 1 1; visual mesh filename=package://Darwin_OP/meshes/shoulder_l.STL scale=1 1 1
- link MP_SHOULDER_R: geometry collision mesh filename=package://Darwin_OP/meshes/shoulder_r_coll.stl scale=1 1 1; visual mesh filename=package://Darwin_OP/meshes/shoulder_r.STL scale=1 1 1
- link MP_THIGH1_L: geometry collision mesh filename=package://Darwin_OP/meshes/thigh1_l_coll.stl scale=1 1 1; visual mesh filename=package://Darwin_OP/meshes/thigh1_l.STL scale=1 1 1
- link MP_THIGH1_R: geometry collision mesh filename=package://Darwin_OP/meshes/thigh1_r_coll.stl scale=1 1 1; visual mesh filename=package://Darwin_OP/meshes/thigh1_r.STL scale=1 1 1
- link MP_THIGH2_L: geometry collision mesh filename=package://Darwin_OP/meshes/thigh2_l_coll.stl scale=1 1 1; visual mesh filename=package://Darwin_OP/meshes/thigh2_l.STL scale=1 1 1
- link MP_THIGH2_R: geometry collision mesh filename=package://Darwin_OP/meshes/thigh2_r_coll.stl scale=1 1 1; visual mesh filename=package://Darwin_OP/meshes/thigh2_r.STL scale=1 1 1
- link MP_TIBIA_L: geometry collision mesh filename=package://Darwin_OP/meshes/tibia_l_coll.stl scale=1 1 1; visual mesh filename=package://Darwin_OP/meshes/tibia_l.STL scale=1 1 1
- link MP_TIBIA_R: geometry collision mesh filename=package://Darwin_OP/meshes/tibia_r_coll.stl scale=1 1 1; visual mesh filename=package://Darwin_OP/meshes/tibia_r.STL scale=1 1 1
